Commit message: feat: describe the payload box in the URDF
The visualiser has always published base_link -> box_link and drawn this mesh
itself, in world coordinates, on the scene topic. The description therefore
described most of a Scout Mini rather than one, and a viewer that loaded it got
a vehicle with no box.

The joint carries the yaw the visualiser applied to the frame and the visual
carries the yaw it applied to the mesh, so the two compose to exactly the pose
the scene used to send. Nothing moves; the box simply now comes from the same
place as the rest of the robot.

Co-Authored-By: Claude Opus 5 (1M context) <noreply@anthropic.com>
Claude-Session: https://claude.ai/code/session_01PTgpaexUo6cTtJmKkbi552

File: urdf/scout_mini.urdf (robot description, URDF)
Before this commit: robot scout_mini, 8 links, 7 joints
Links:
- added link box_link; visual mesh filename=package://scout_description/meshes/box_link.STL
Joints:
- added joint box_joint: type fixed, parent base_link, child box_link, origin xyz=0 0 0.055 rpy=0 0 3.14
